File: Regulated Board/Regulated Board.kicad_pcb (KiCad board)
At the start: 2 copper layers, 0 parts

Commit message: Added a lot of footprints and did some PCB layout
Need to find footprints and appropriate screw terminals. Will route.
Parts:
- added C1: 2.2uF, Capacitor_THT:CP_Radial_D5.0mm_P2.00mm, F.Cu at (108.5, -43.0)
- added C2: 2.2uF, Capacitor_THT:CP_Radial_D5.0mm_P2.00mm, F.Cu at (102.0, -43.0)
- added C3: 2.2uF, Capacitor_THT:CP_Radial_D5.0mm_P2.00mm, F.Cu at (95.4, -43.0)
- added F1: Fuse, Library:FUSE_3544-2, F.Cu at (-41.7, -409.5)
- added F10: Fuse, Library:FUSE_3544-2, F.Cu at (-41.7, -316.6)
- added F100: Fuse, Library:FUSE_3544-2, F.Cu at (31.8, -212.9)
- added F101: Fuse, Library:FUSE_3544-2, F.Cu at (31.8, -202.6)
- added F102: Fuse, Library:FUSE_3544-2, F.Cu at (31.8, -192.2)
- added F103: Fuse, Library:FUSE_3544-2, F.Cu at (31.8, -181.9)
- added F104: Fuse, Library:FUSE_3544-2, F.Cu at (31.8, -171.5)
- added F105: Fuse, Library:FUSE_3544-2, F.Cu at (31.8, -161.2)
- added F106: Fuse, Library:FUSE_3544-2, F.Cu at (31.8, -150.8)
- added F107: Fuse, Library:FUSE_3544-2, F.Cu at (31.8, -140.5)
- added F108: Fuse, Library:FUSE_3544-2, F.Cu at (31.8, -130.2)
- added F109: Fuse, Library:FUSE_3544-2, F.Cu at (31.8, -119.8)
- added F11: Fuse, Library:FUSE_3544-2, F.Cu at (-41.7, -306.3)
- added F110: Fuse, Library:FUSE_3544-2, F.Cu at (31.8, -109.5)
- added F111: Fuse, Library:FUSE_3544-2, F.Cu at (31.8, -99.1)
- added F112: Fuse, Library:FUSE_3544-2, F.Cu at (31.8, -88.8)
- added F113: Fuse, Library:FUSE_3544-2, F.Cu at (31.8, -78.4)
- added F114: Fuse, Library:FUSE_3544-2, F.Cu at (31.8, -68.1)
- added F115: Fuse, Library:FUSE_3544-2, F.Cu at (31.8, -57.7)
- added F116: Fuse, Library:FUSE_3544-2, F.Cu at (31.8, -47.4)
- added F117: Fuse, Library:FUSE_3544-2, F.Cu at (31.8, -37.0)
- added F118: Fuse, Library:FUSE_3544-2, F.Cu at (31.8, -26.7)
- added F119: Fuse, Library:FUSE_3544-2, F.Cu at (31.8, -16.3)
- added F12: Fuse, Library:FUSE_3544-2, F.Cu at (-41.7, -295.9)
- added F120: Fuse, Library:FUSE_3544-2, F.Cu at (31.8, -6.00)
- added F121: Fuse, Library:FUSE_3544-2, F.Cu at (102.3, -31.9)
- added F122: Fuse, Library:FUSE_3544-2, F.Cu at (102.3, -23.9)
- added F123: Fuse, Library:FUSE_3544-2, F.Cu at (102.3, -16.0)
- added F124: Fuse, Library:FUSE_3544-2, F.Cu at (102.3, -8.05)
- added F13: Fuse, Library:FUSE_3544-2, F.Cu at (-41.7, -285.6)
- added F14: Fuse, Library:FUSE_3544-2, F.Cu at (-41.7, -275.3)
- added F15: Fuse, Library:FUSE_3544-2, F.Cu at (-41.7, -265.0)
- added F16: Fuse, Library:FUSE_3544-2, F.Cu at (-41.7, -254.7)
- added F17: Fuse, Library:FUSE_3544-2, F.Cu at (-41.7, -244.3)
- added F18: Fuse, Library:FUSE_3544-2, F.Cu at (-41.7, -234.0)
- added F19: Fuse, Library:FUSE_3544-2, F.Cu at (-41.7, -223.7)
- added F2: Fuse, Library:FUSE_3544-2, F.Cu at (-41.7, -399.2)
- added F20: Fuse, Library:FUSE_3544-2, F.Cu at (-41.7, -213.4)
- added F21: Fuse, Library:FUSE_3544-2, F.Cu at (-41.7, -203.0)
- added F22: Fuse, Library:FUSE_3544-2, F.Cu at (-41.7, -192.7)
- added F23: Fuse, Library:FUSE_3544-2, F.Cu at (-41.7, -182.4)
- added F24: Fuse, Library:FUSE_3544-2, F.Cu at (-41.7, -172.1)
- added F25: Fuse, Library:FUSE_3544-2, F.Cu at (-41.7, -161.7)
- added F26: Fuse, Library:FUSE_3544-2, F.Cu at (-41.7, -151.4)
- added F27: Fuse, Library:FUSE_3544-2, F.Cu at (-41.7, -141.1)
- added F28: Fuse, Library:FUSE_3544-2, F.Cu at (-41.7, -130.8)
- added F29: Fuse, Library:FUSE_3544-2, F.Cu at (-41.7, -120.5)
- added F3: Fuse, Library:FUSE_3544-2, F.Cu at (-41.7, -388.9)
- added F30: Fuse, Library:FUSE_3544-2, F.Cu at (-41.7, -110.1)
- added F31: Fuse, Library:FUSE_3544-2, F.Cu at (-41.7, -99.8)
- added F32: Fuse, Library:FUSE_3544-2, F.Cu at (-41.7, -89.5)
- added F33: Fuse, Library:FUSE_3544-2, F.Cu at (-41.7, -79.2)
- added F34: Fuse, Library:FUSE_3544-2, F.Cu at (-41.7, -68.8)
- added F35: Fuse, Library:FUSE_3544-2, F.Cu at (-41.7, -58.5)
- added F36: Fuse, Library:FUSE_3544-2, F.Cu at (-41.7, -48.2)
- added F37: Fuse, Library:FUSE_3544-2, F.Cu at (-41.7, -37.9)
- added F38: Fuse, Library:FUSE_3544-2, F.Cu at (-41.7, -27.5)
- added F39: Fuse, Library:FUSE_3544-2, F.Cu at (-41.7, -17.2)
- added F4: Fuse, Library:FUSE_3544-2, F.Cu at (-41.7, -378.5)
- added F40: Fuse, Library:FUSE_3544-2, F.Cu at (-41.7, -6.90)
- added F41: Fuse, Library:FUSE_3544-2, F.Cu at (-4.70, -409.5)
- added F42: Fuse, Library:FUSE_3544-2, F.Cu at (-4.70, -399.2)
- added F43: Fuse, Library:FUSE_3544-2, F.Cu at (-4.70, -388.8)
- added F44: Fuse, Library:FUSE_3544-2, F.Cu at (-4.70, -378.5)
- added F45: Fuse, Library:FUSE_3544-2, F.Cu at (-4.70, -368.1)
- added F46: Fuse, Library:FUSE_3544-2, F.Cu at (-4.70, -357.8)
- added F47: Fuse, Library:FUSE_3544-2, F.Cu at (-4.70, -347.5)
- added F48: Fuse, Library:FUSE_3544-2, F.Cu at (-4.70, -337.1)
- added F49: Fuse, Library:FUSE_3544-2, F.Cu at (-4.70, -326.8)
- added F5: Fuse, Library:FUSE_3544-2, F.Cu at (-41.7, -368.2)
- added F50: Fuse, Library:FUSE_3544-2, F.Cu at (-4.70, -316.4)
- added F51: Fuse, Library:FUSE_3544-2, F.Cu at (-4.70, -306.1)
- added F52: Fuse, Library:FUSE_3544-2, F.Cu at (-4.70, -295.8)
- added F53: Fuse, Library:FUSE_3544-2, F.Cu at (-4.70, -285.4)
- added F54: Fuse, Library:FUSE_3544-2, F.Cu at (-4.70, -275.1)
- added F55: Fuse, Library:FUSE_3544-2, F.Cu at (-4.70, -264.7)
- added F56: Fuse, Library:FUSE_3544-2, F.Cu at (-4.70, -254.4)
- added F57: Fuse, Library:FUSE_3544-2, F.Cu at (-4.70, -244.1)
- added F58: Fuse, Library:FUSE_3544-2, F.Cu at (-4.70, -233.7)
- added F59: Fuse, Library:FUSE_3544-2, F.Cu at (-4.70, -223.4)
- added F6: Fuse, Library:FUSE_3544-2, F.Cu at (-41.7, -357.9)
- added F60: Fuse, Library:FUSE_3544-2, F.Cu at (-4.70, -213.0)
- added F61: Fuse, Library:FUSE_3544-2, F.Cu at (-4.70, -202.7)
- added F62: Fuse, Library:FUSE_3544-2, F.Cu at (-4.70, -192.4)
- added F63: Fuse, Library:FUSE_3544-2, F.Cu at (-4.70, -182.0)
- added F64: Fuse, Library:FUSE_3544-2, F.Cu at (-4.70, -171.7)
- added F65: Fuse, Library:FUSE_3544-2, F.Cu at (-4.70, -161.3)
- added F66: Fuse, Library:FUSE_3544-2, F.Cu at (-4.70, -151.0)
- added F67: Fuse, Library:FUSE_3544-2, F.Cu at (-4.70, -140.7)
- added F68: Fuse, Library:FUSE_3544-2, F.Cu at (-4.70, -130.3)
- added F69: Fuse, Library:FUSE_3544-2, F.Cu at (-4.70, -120.0)
- added F7: Fuse, Library:FUSE_3544-2, F.Cu at (-41.7, -347.6)
- added F70: Fuse, Library:FUSE_3544-2, F.Cu at (-4.70, -109.6)
- added F71: Fuse, Library:FUSE_3544-2, F.Cu at (-4.70, -99.3)
- added F72: Fuse, Library:FUSE_3544-2, F.Cu at (-4.70, -89.0)
- added F73: Fuse, Library:FUSE_3544-2, F.Cu at (-4.70, -78.6)
- added F74: Fuse, Library:FUSE_3544-2, F.Cu at (-4.70, -68.3)
- added F75: Fuse, Library:FUSE_3544-2, F.Cu at (-4.70, -57.9)
- added F76: Fuse, Library:FUSE_3544-2, F.Cu at (-4.70, -47.6)
- added F77: Fuse, Library:FUSE_3544-2, F.Cu at (-4.70, -37.3)
- added F78: Fuse, Library:FUSE_3544-2, F.Cu at (-4.70, -26.9)
- added F79: Fuse, Library:FUSE_3544-2, F.Cu at (-4.70, -16.6)
- added F8: Fuse, Library:FUSE_3544-2, F.Cu at (-41.7, -337.2)
- added F80: Fuse, Library:FUSE_3544-2, F.Cu at (-4.70, -6.25)
- added F81: Fuse, Library:FUSE_3544-2, F.Cu at (31.8, -409.5)
- added F82: Fuse, Library:FUSE_3544-2, F.Cu at (31.8, -399.2)
- added F83: Fuse, Library:FUSE_3544-2, F.Cu at (31.8, -388.8)
- added F84: Fuse, Library:FUSE_3544-2, F.Cu at (31.8, -378.5)
- added F85: Fuse, Library:FUSE_3544-2, F.Cu at (31.8, -368.1)
- added F86: Fuse, Library:FUSE_3544-2, F.Cu at (31.8, -357.8)
- added F87: Fuse, Library:FUSE_3544-2, F.Cu at (31.8, -347.4)
- added F88: Fuse, Library:FUSE_3544-2, F.Cu at (31.8, -337.1)
- added F89: Fuse, Library:FUSE_3544-2, F.Cu at (31.8, -326.7)
- added F9: Fuse, Library:FUSE_3544-2, F.Cu at (-41.7, -326.9)
- added F90: Fuse, Library:FUSE_3544-2, F.Cu at (31.8, -316.4)
- added F91: Fuse, Library:FUSE_3544-2, F.Cu at (31.8, -306.0)
- added F92: Fuse, Library:FUSE_3544-2, F.Cu at (31.8, -295.7)
- added F93: Fuse, Library:FUSE_3544-2, F.Cu at (31.8, -285.3)
- added F94: Fuse, Library:FUSE_3544-2, F.Cu at (31.8, -275.0)
- added F95: Fuse, Library:FUSE_3544-2, F.Cu at (31.8, -264.7)
- added F96: Fuse, Library:FUSE_3544-2, F.Cu at (31.8, -254.3)
- added F97: Fuse, Library:FUSE_3544-2, F.Cu at (31.8, -244.0)
- added F98: Fuse, Library:FUSE_3544-2, F.Cu at (31.8, -233.6)
- added F99: Fuse, Library:FUSE_3544-2, F.Cu at (31.8, -223.3)
- added J1: Screw_Terminal_01x02, Connector_PinHeader_2.54mm:PinHeader_1x02_P2.54mm_Vertical, F.Cu at (123.0, -34.5)
- added J10: Screw_Terminal_01x02, Connector_PinHeader_2.54mm:PinHeader_1x02_P2.54mm_Vertical, F.Cu at (123.0, -11.2)
- added J13: Screw_Terminal_01x02, Connector_PinHeader_2.54mm:PinHeader_1x02_P2.54mm_Vertical, F.Cu at (123.0, -6.55)
- added J14: Conn_01x01, Connector_PinHeader_2.54mm:PinHeader_1x01_P2.54mm_Vertical, F.Cu at (144.1, -25.1)
- added J15: Conn_01x01, Connector_PinHeader_2.54mm:PinHeader_1x01_P2.54mm_Vertical, F.Cu at (144.1, -20.4)
- added J16: Conn_01x01, Connector_PinHeader_2.54mm:PinHeader_1x01_P2.54mm_Vertical, F.Cu at (144.1, -15.8)
- added J2: Screw_Terminal_01x02, Connector_PinHeader_2.54mm:PinHeader_1x02_P2.54mm_Vertical, F.Cu at (123.0, -29.8)
- added J4: Screw_Terminal_01x02, Connector_PinHeader_2.54mm:PinHeader_1x02_P2.54mm_Vertical, F.Cu at (123.0, -25.1)
- added J5: Screw_Terminal_01x02, Connector_PinHeader_2.54mm:PinHeader_1x02_P2.54mm_Vertical, F.Cu at (123.0, -20.5)
- added J6: Screw_Terminal_01x02, Connector_PinHeader_2.54mm:PinHeader_1x02_P2.54mm_Vertical, F.Cu at (123.0, -15.8)
- added L1: TCK, Library:TCK-076, F.Cu at (152.4, -41.4)
- added L2: TCK, Library:TCK-076, F.Cu at (154.3, -5.32)
- added Q1: IRLZ44N, Package_TO_SOT_THT:TO-220-3_Vertical, F.Cu at (133.4, -23.5)
- added Q3: IRLZ44N, Package_TO_SOT_THT:TO-220-3_Vertical, F.Cu at (133.4, -17.5)
- added Q4: IRLZ44N, Package_TO_SOT_THT:TO-220-3_Vertical, F.Cu at (133.4, -11.5)
Routing:
- net Net-(J9-Pin_7): vias 0 -> 1
- net Net-(J9-Pin_20): vias 0 -> 1
- net Net-(J9-Pin_19): vias 0 -> 1
- net Net-(J9-Pin_18): vias 0 -> 1
- net Net-(J9-Pin_17): vias 0 -> 1
- net Net-(J9-Pin_16): vias 0 -> 1
- net Net-(J9-Pin_14): vias 0 -> 1
- net Net-(J9-Pin_13): vias 0 -> 1
- net Net-(J9-Pin_12): vias 0 -> 1
- net Net-(J9-Pin_11): vias 0 -> 2
- net Net-(J8-Pin_7): vias 0 -> 1
- net Net-(J8-Pin_5): vias 0 -> 1
- net Net-(J8-Pin_2): vias 0 -> 1
- net Net-(J8-Pin_13): vias 0 -> 1
- net Net-(J8-Pin_12): vias 0 -> 1
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Other:
- board outline added: 254 x 442 mm
