File: RFD900TestBoard/pcblunarroverrfd900x modem.kicad_sch (KiCad schematic)
At the start: 0 parts

Commit message: edits
Parts:
- added J1: Barrel_Jack, Connector_BarrelJack:BarrelJack_SwitchcraftConxall_RAPC10U_Horizontal, symbol Connector:Barrel_Jack
- added J2: Conn_02x08_Counter_Clockwise, Connector_DIN:DIN41612_B2_2x8_Male_Horizontal_THT, symbol Connector_Generic:Conn_02x08_Counter_Clockwise
- added U1: ESP32-DEVKIT-V1, hi:MODULE_ESP32_DEVKIT_V1, symbol ESP32-DEVKIT-V1:ESP32-DEVKIT-V1
- added U2: GPS-15136, hi:MODULE_GPS-15136, symbol GPS-15136:GPS-15136
Connections:
- new net +3.3V: U1.1 (3V3), U2.J1_4 (3.3V_J1)
- new net +5V: J1.1, J2.15 (Pin_15), U1.30 (VIN)
- new net CTS: J2.2 (Pin_2), U1.14 (D22)
- new net GND: J1.2, J2.1 (Pin_1), U1.2 (GND), U1.29 (GND), U2.J1_6 (GND_J1)
- new net INT: U1.8 (D5), U2.J6_6 (INT)
- new net RESET: U1.4 (D2), U2.J6_4 (~{RESET})
- new net RTS: J2.6 (Pin_6), U1.15 (D23)
- new net RX: J2.4 (Pin_4), U1.13 (TX0)
- new net RX2: U1.7 (TX2), U2.J1_3 (RX2_J1)
- new net SAFE: U1.5 (D4), U2.J6_5 (~{SAFE})
- new net TX: J2.5 (Pin_5), U1.12 (RX0)
- new net TX2: U1.6 (RX2), U2.J1_2 (TX2_J1)

Commit message: edits
Parts:
- added R1, R2, R3, R4: R, Resistor_THT:R_Axial_DIN0204_L3.6mm_D1.6mm_P1.90mm_Vertical, symbol Device:R
Connections:
- net +3.3V: now also U2.J7_7 (3.3V_J7)
- net CTS: now also U1.27 (D12), R1.1; no longer J2.2 (Pin_2), U1.14 (D22)
- net GND: now also U2.J7_9 (GND_J7)
- net RTS: now also R4.1; no longer J2.6 (Pin_6)
- net RX: now also R2.1; no longer J2.4 (Pin_4)
- net TX: now also R3.1; no longer J2.5 (Pin_5)
- net SCL: now reaches U2.J7_1 (SCL/SCK_J7)
- net SCL: now also U1.14 (D22)
- net SDA: now reaches U2.J7_4 (SDA/~{CS}_J7)
- net SDA: now also U1.11 (D21)
- new net: J2.5 (Pin_5), R3.2
- new net: J2.2 (Pin_2), R1.2
- new net: J2.4 (Pin_4), R2.2
- new net: J2.6 (Pin_6), R4.2

Commit message: made changes to RFD900x test board
Parts:
- R1, R2, R3, R4: value R -> 1k; footprint Resistor_THT:R_Axial_DIN0204_L3.6mm_D1.6mm_P1.90mm_Vertical -> \
Connections:
- net RESET renamed RST
Other:
- note added: "ESP32 Controller"
- note added: "GNSS Module"
- note added: "Power"
- note added: "RFD900x Housing Board"
- note added: "RFD900x Pin Header Connection"
- moved on the sheet: J1, J2, R1, U1, U2A, U2B, U2C, U2D
