File: RFD900TestBoard/pcblunarroverrfd900x modem.kicad_pcb (KiCad board)
At the start: 4 copper layers, 135 x 89.4 mm, 27 parts, among them J1 Barrel_Jack_Switch, J10 Conn_02x01, J11 Conn_02x01, J12 Conn_02x01, J13 Conn_02x01, J14 Conn_02x01, J16 Conn_02x01, J17 Conn_02x01, J18 Conn_01x11, J2 Conn_02x08_Counter_Clockwise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

Commit message: panelized rfd and motor controller pcb for ordering
Parts:
- added D1: LED, LED_THT:LED_D5.0mm, F.Cu at (252.0, 38.5)
- added J1: DC-005-5A-2.0, DC-005-5A-2.0:XKB_DC-005-5A-2.0, F.Cu at (227.0, 35.0)
- added J2: Conn_01x01_Pin, Connector_PinHeader_2.54mm:PinHeader_1x01_P2.54mm_Vertical, F.Cu at (247.0, 29.5)
- added J4: Conn_01x10_Socket, Connector_PinHeader_2.54mm:PinHeader_1x10_P2.54mm_Vertical, F.Cu at (216.5, 87.8)
- added J5: Conn_01x03_Socket, Connector_PinHeader_2.54mm:PinHeader_1x03_P2.54mm_Vertical, F.Cu at (254.0, 70.0)
- added J6: Conn_01x02_Socket, Connector_PinHeader_2.54mm:PinHeader_1x02_P2.54mm_Vertical, F.Cu at (220.0, 95.3)
- added J7: Conn_01x03_Pin, Connector_PinHeader_2.54mm:PinHeader_1x03_P2.54mm_Vertical, F.Cu at (236.0, 34.5)
- added MC1: Conn_02x04_Counter_Clockwise, ModifiedFootprints:16_pin_custom_wraparound_connector, F.Cu at (179.7, 34.2)
- added MC2: Conn_02x04_Counter_Clockwise, ModifiedFootprints:16_pin_custom_wraparound_connector, F.Cu at (205.5, 34.0)
- added MC3: Conn_02x04_Counter_Clockwise, ModifiedFootprints:16_pin_custom_wraparound_connector, F.Cu at (205.6, 120.2)
- added MC4: Conn_02x04_Counter_Clockwise, ModifiedFootprints:16_pin_custom_wraparound_connector, F.Cu at (173.3, 75.2)
- added MC5: Conn_02x04_Counter_Clockwise, ModifiedFootprints:16_pin_custom_wraparound_connector, F.Cu at (180.1, 120.2)
- added OLED1: Conn_01x04, Connector_PinHeader_2.54mm:PinHeader_1x04_P2.54mm_Vertical, F.Cu at (249.0, 110.9)
- added R1: R_Small_US, Resistor_THT:R_Axial_DIN0204_L3.6mm_D1.6mm_P2.54mm_Vertical, F.Cu at (224.3, 123.0)
- added R2: R_Small_US, Resistor_THT:R_Axial_DIN0204_L3.6mm_D1.6mm_P2.54mm_Vertical, F.Cu at (224.3, 120.5)
- added R3: R_Small_US, Connector_PinHeader_2.54mm:PinHeader_1x02_P2.54mm_Vertical, F.Cu at (241.2, 47.0)
- added R4: R_Small_US, Connector_PinHeader_2.54mm:PinHeader_1x02_P2.54mm_Vertical, F.Cu at (234.5, 47.0)
- added R5: R_Small_US, Connector_PinHeader_2.54mm:PinHeader_1x02_P2.54mm_Vertical, F.Cu at (250.7, 43.0)
- added RE1: Conn_01x04, Connector_PinHeader_2.54mm:PinHeader_1x04_P2.54mm_Vertical, F.Cu at (170.0, 48.7)
- added RE2: Conn_01x04, Connector_PinHeader_2.54mm:PinHeader_1x04_P2.54mm_Vertical, F.Cu at (197.5, 48.7)
- added RE3: Conn_01x04, Connector_PinHeader_2.54mm:PinHeader_1x04_P2.54mm_Vertical, F.Cu at (211.5, 102.1)
- added RE4: Conn_01x04, Connector_PinHeader_2.54mm:PinHeader_1x04_P2.54mm_Vertical, F.Cu at (205.5, 76.0)
- added RE5: Conn_01x04, Connector_PinHeader_2.54mm:PinHeader_1x04_P2.54mm_Vertical, F.Cu at (187.5, 102.8)
- added SW1: MAX11617, SerialWombat:sw_pcb0029, F.Cu at (186.1, 52.2)
- added SW2: MAX11617, SerialWombat:sw_pcb0029, F.Cu at (212.8, 51.7)
- added SW3: MAX11617, SerialWombat:sw_pcb0029, F.Cu at (198.7, 100.8)
- added SW4: MAX11617, SerialWombat:sw_pcb0029, F.Cu at (187.7, 76.0)
- added SW5: MAX11617, SerialWombat:sw_pcb0029, F.Cu at (171.7, 100.5)
- added U1: ESP32-DEVKIT-V1, ESP32-DEVKIT-V1:MODULE_ESP32_DEVKIT_V1, F.Cu at (236.5, 77.2)
- added U3: L7805, Connector_PinHeader_2.54mm:PinHeader_1x03_P2.54mm_Vertical, F.Cu at (236.0, 29.5)
- moved 10uF2 48.0 mm to (92.4, 58.0)
- moved 0.1uF3 48.0 mm to (127.8, 39.3)
- moved 0.1uf2 48.0 mm to (100.6, 58.0)
- moved 1000uf1 48.0 mm to (35.6, 94.5)
- moved 10uF1 48.0 mm to (127.8, 47.0)
- moved 1k 48.0 mm to (138.2, 97.8)
- moved D1 48.0 mm to (145.9, 99.1)
- moved J1 48.0 mm to (154.1, 44.6)
- moved J10 48.0 mm to (40.0, 41.4)
- moved J11 48.0 mm to (116.1, 45.2)
- moved J13 48.0 mm to (97.6, 81.1)
- moved J14 48.0 mm to (92.5, 81.2)
- moved J16 48.0 mm to (92.5, 88.6)
- moved J17 48.0 mm to (97.6, 88.5)
- moved J18 48.0 mm to (27.1, 40.7)
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Routing:
- net SCL: track 53.2 -> 291.3 mm, vias 0 -> 4
- net SDA: track 46.2 -> 277.7 mm, vias 0 -> 5
- net 3.3V: track 0.00 -> 49.6 mm, vias 0 -> 1
- net Net-(U1-D2): track 0.00 -> 46.2 mm
- net Net-(MC5-Pin_6): track 0.00 -> 32.2 mm
- net Net-(MC5-Pin_4): track 0.00 -> 29.4 mm
- net Net-(MC3-Pin_4): track 0.00 -> 27.8 mm
- net Net-(MC3-Pin_3): track 0.00 -> 24.0 mm
- net Net-(MC2-Pin_7): track 0.00 -> 23.1 mm
- net Net-(MC1-Pin_7): track 0.00 -> 22.6 mm
- net Net-(MC4-Pin_3): track 0.00 -> 22.2 mm
- net Net-(MC4-Pin_2): track 0.00 -> 21.9 mm
- net Net-(MC5-Pin_7): track 0.00 -> 21.7 mm, vias 0 -> 1
- net Net-(MC5-Pin_5): track 0.00 -> 21.4 mm
- net Net-(MC3-Pin_7): track 0.00 -> 20.2 mm
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- added copper zone on In2.Cu, net 5V
- added copper zone on In2.Cu, net ESP32Feeder
- added copper zone on B.Cu, net GND
- added copper zone on F.Cu, net GND
- added copper zone on In2.Cu, net Vin
Other:
- board size 135 x 89.4 mm -> 238 x 100.1 mm
- board text added: "12V 5V"
- board text added: "5V"
- board text added: "<< I2C Pull-ups"
- board text added: "Connect these to power ESP-32 using 5V battery, not USB port >>"
- board text added: "GND 5V"
- board text added: "IN"
- board text added: "L7805"
- board text added: "LED"
- board text added: "M0 DRILL"
- board text added: "M1 DTRF"
- board text added: "M2 DTRB"
- board text added: "M3 DTLB"
- board text added: "M4 DTLF"
- board text added: "OUT"
- board text added: "Power?"
- board text added: "R1"
- board text added: "R2"
- board text added: "SW 0000"
- board text added: "SW 0001"
- board text added: "SW 0010"
- board text added: "SW 0011"
- board text added: "SW 0100"
- board text added: "SW0: R_IS SW1: R_EN SW2: R_PWM SW3: L_PWM SW4: L_EN SW5: R_IS SW6: RE CH A SW7: RE CH B"
- board text added: "Write D15 {dblquote}HIGH{dblquote} to cut off power to SW chips, motors, & REs. Read voltage level at D23 & multiply by appropriate factor _____ to get voltage level of battery."
- board text added: "inside +5V, outside GND >>"
- board text added: "make one of these connections based on battery voltage"
- board text added: "resistor"
- board text added: "voltage divider resistors"
- board text added: "~Rover ELEC 2025-26 :D"
