File: DrivetrainDrillMotorControllerPCB/DrivetrainDrillMotorControllerPCB.kicad_pcb (KiCad board)
At the start: 4 copper layers, 100 x 100 mm, 42 parts, among them J1 DC-005-5A-2.0, J10 Conn_01x02_Socket, J11 Conn_01x02_Socket, J12 Conn_01x02_Socket, J13 Conn_01x02_Socket, J14 Conn_01x02_Socket, J15 Conn_01x02_Socket, J16 Conn_01x02_Socket, J2 Conn_01x02_Socket, J3 Conn_01x02_Socket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

Commit message: Final
Connections:
- R1 pad 2: original5V -> 3.3V
- R2 pad 2: original5V -> 3.3V
Routing:
- net 3.3V: track 22.0 -> 49.6 mm
Changed lines of the file:
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@@
 			(layers "*.Cu" "*.Mask")
 			(remove_unused_layers no)
-			(net 82 "original5V")
+			(net 93 "3.3V")
 			(pintype "passive")
 		)
@@
 			(layers "*.Cu" "*.Mask")
 			(remove_unused_layers no)
-			(net 82 "original5V")
+			(net 93 "3.3V")
 			(pintype "passive")
 		)
@@
 	)
 	(segment
+		(start 146.5 147.42)
+		(end 139.42 154.5)
+		(width 0.2)
+		(layer "B.Cu")
+		(net 93)
+	)
+	(segment
+		(start 124.32 154.5)
+		(end 124.32 157)
+		(width 0.2)
+		(layer "B.Cu")
+		(net 93)
+	)
+	(segment
+		(start 139.42 154.5)
+		(end 124.32 154.5)
+		(width 0.2)
+		(layer "B.Cu")
+		(net 93)
+	)
+	(segment
 		(start 114 109.08)
 		(end 121.155 109.08)
@@
 		(polygon
 			(pts
-				(xy 57.5 60) (xy 117 60) (xy 117 79.5) (xy 127 79.5) (xy 127 79.5) (xy 123.5 79.5) (xy 123.5 86.279599)
-				(xy 115.010208 92.898232) (xy 115.500001 160) (xy 57.5 160)
+				(xy 57.5 60) (xy 117 60) (xy 117 79.5) (xy 127 79.5) (xy 123.5 79.5) (xy 123.5 86.279599) (xy 115.010208 92.898232)
+				(xy 115.500001 160) (xy 57.5 160)
 			)
 		)

Commit message: Added GND pin, connected REs to SW
Parts:
- removed J10, J11, J12, J13, J14, J15, J16, J2, J3, J9: Conn_01x02_Socket, Connector_PinHeader_2.54mm:PinHeader_1x02_P2.54mm_Vertical
- added GND: Conn_01x01_Pin, Connector_PinHeader_2.54mm:PinHeader_1x01_P2.54mm_Vertical, F.Cu at (144.5, 63.5)
- moved RE3 56.3 mm to (84.5, 136.8), turned to 180 degrees
- moved RE4 56.0 mm to (68.0, 82.7), turned to 0 degrees
- moved RE2 3.51 mm to (109.0, 136.3)
- moved RE1 0.50 mm to (102.5, 111.3)
Connections:
- RE1 pad 3: Net-(J2-Pin_2) -> Net-(RE1-Pin_3)
- RE1 pad 4: Net-(J2-Pin_1) -> Net-(RE1-Pin_4)
- RE2 pad 3: Net-(J9-Pin_2) -> Net-(RE2-Pin_3)
- RE2 pad 4: Net-(J9-Pin_1) -> Net-(RE2-Pin_4)
- RE3 pad 3: Net-(J11-Pin_2) -> Net-(RE3-Pin_3)
- RE3 pad 4: Net-(J11-Pin_1) -> Net-(RE3-Pin_4)
- RE4 pad 3: Net-(J13-Pin_2) -> Net-(RE4-Pin_3)
- RE4 pad 4: Net-(J13-Pin_1) -> Net-(RE4-Pin_4)
- RE5 pad 3: Net-(J15-Pin_2) -> Net-(RE5-Pin_3)
- RE5 pad 4: Net-(J15-Pin_1) -> Net-(RE5-Pin_4)
- SW1 pad 11: Net-(J3-Pin_2) -> Net-(RE1-Pin_3)
- SW1 pad 12: Net-(J3-Pin_1) -> Net-(RE1-Pin_4)
- SW2 pad 11: Net-(J10-Pin_2) -> Net-(RE2-Pin_3)
- SW2 pad 12: Net-(J10-Pin_1) -> Net-(RE2-Pin_4)
- SW3 pad 11: Net-(J12-Pin_2) -> Net-(RE3-Pin_3)
- SW3 pad 12: Net-(J12-Pin_1) -> Net-(RE3-Pin_4)
- SW4 pad 11: Net-(J14-Pin_2) -> Net-(RE4-Pin_3)
- SW4 pad 12: Net-(J14-Pin_1) -> Net-(RE4-Pin_4)
- SW5 pad 11: Net-(J16-Pin_2) -> Net-(RE5-Pin_3)
- SW5 pad 12: Net-(J16-Pin_1) -> Net-(RE5-Pin_4)
Routing:
- net Net-(RE1-Pin_4): track 0.00 -> 18.3 mm
- net Net-(RE1-Pin_3): track 0.00 -> 18.2 mm
- net Net-(RE4-Pin_4): track 0.00 -> 14.9 mm
- net Net-(RE4-Pin_3): track 0.00 -> 14.9 mm
- net Net-(RE3-Pin_4): track 0.00 -> 14.8 mm
- net Net-(RE3-Pin_3): track 0.00 -> 14.8 mm
- net Net-(RE5-Pin_3): track 0.00 -> 14.8 mm
- net Net-(RE5-Pin_4): track 0.00 -> 14.7 mm
- net Net-(RE2-Pin_4): track 0.00 -> 12.7 mm
- net Net-(RE2-Pin_3): track 0.00 -> 12.6 mm
- net Net-(J2-Pin_2): track 7.64 -> 0.00 mm
- net Net-(J2-Pin_1): track 7.64 -> 0.00 mm
- net Net-(J11-Pin_2): track 7.11 -> 0.00 mm
- net Net-(J11-Pin_1): track 7.11 -> 0.00 mm
- net Net-(J9-Pin_2): track 7.01 -> 0.00 mm
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Other:
- board text added: "SW0: R_IS SW1: R_EN SW2: R_PWM SW3: L_PWM SW4: L_EN SW5: R_IS SW6: RE CH A SW7: RE CH B"
- board text removed: "D34: CLK2 D35: DT2 D32: CLK1 D33: DT1 D25: CLK0 D26: DT0 D27: CLK4 D14: DT4 D12: CLK3 D13: DT3"
- board text removed: "SW1: R_IS SW2: R_EN SW3: R_PWM SW4: L_PWM SW5: L_EN SW6: R_IS SW7: CLK SW8: DT"

Commit message: Misc motor control pcb stuff
Parts:
- removed 100k1: R_Small_US, Connector_PinHeader_2.54mm:PinHeader_1x02_P2.54mm_Vertical
- removed Q1: PMOS, Connector_PinHeader_2.54mm:PinHeader_1x03_P2.54mm_Vertical
- removed Q2: NMOS, Connector_PinHeader_2.54mm:PinHeader_1x03_P2.54mm_Vertical
- MC1, MC2, MC3, MC4, MC5: footprint Connector_IDC:IDC-Header_2x04_P2.54mm_Vertical -> ModifiedFootprints:16_pin_custom_wraparound_connector
- moved MC5 92.7 mm to (77.6, 154.2), turned to 90 degrees
- moved MC2 87.0 mm to (103.0, 68.0)
- moved SW5 63.8 mm to (69.2, 134.5), turned to 0 degrees
- moved RE2 55.4 mm to (95.0, 82.7), turned to 0 degrees
- moved RE5 54.8 mm to (85.0, 136.8), turned to 180 degrees
- moved SW2 51.2 mm to (110.3, 85.7), turned to 180 degrees
- moved RE1 45.2 mm to (67.5, 82.7), turned to 0 degrees
- moved RE4 44.4 mm to (103.0, 110.0), turned to 180 degrees
- moved MC4 44.1 mm to (70.8, 109.2), turned to 0 degrees
- moved MC1 38.5 mm to (77.2, 68.2), turned to 90 degrees
- moved MC3 29.3 mm to (103.1, 154.2)
- moved SW3 26.8 mm to (96.2, 134.8)
- moved SW1 24.5 mm to (83.6, 86.2), turned to 180 degrees
- moved RE3 24.5 mm to (109.0, 136.1)
- moved SW4 24.4 mm to (85.2, 110.0), turned to 0 degrees
- renumbered GND to J2
Connections:
- D1 pad 2: original5V -> 5V
- J6 pad 1: original5V -> 5V
- J7 pad 3: original5V -> 5V
- SW1 pad 13: SCL -> SDA
- SW1 pad 14: SDA -> SCL
- SW1 pad 15: GND -> 5V
- SW1 pad 16: 5V -> GND
- SW2 pad 13: SCL -> SDA
- SW2 pad 14: SDA -> SCL
- SW2 pad 15: GND -> 5V
- SW2 pad 16: 5V -> GND
- SW3 pad 13: SCL -> SDA
- SW3 pad 14: SDA -> SCL
- SW3 pad 15: GND -> 5V
- SW3 pad 16: 5V -> GND
- SW4 pad 13: SCL -> SDA
- SW4 pad 14: SDA -> SCL
- SW4 pad 15: GND -> 5V
- SW4 pad 16: 5V -> GND
- SW5 pad 13: SCL -> SDA
- SW5 pad 14: SDA -> SCL
- SW5 pad 15: GND -> 5V
- SW5 pad 16: 5V -> GND
- U1 pad 3: Net-(Q2-G) -> unconnected-(U1-D15-Pad3)
- U3 pad 3: original5V -> 5V
Routing:
- net Net-(Q2-G): track 69.0 -> 0.00 mm
- net Net-(Q1-G): track 32.3 -> 0.00 mm, vias 1 -> 0
- net Net-(MC1-Pin_3): track 30.9 -> 8.41 mm
- net Net-(MC1-Pin_2): track 32.6 -> 12.0 mm
- net Net-(MC5-Pin_4): track 12.2 -> 29.4 mm
- net Net-(MC5-Pin_6): track 17.8 -> 32.2 mm
- net Net-(MC4-Pin_7): track 24.0 -> 10.1 mm
- net Net-(MC3-Pin_4): track 14.4 -> 27.8 mm
- net Net-(MC4-Pin_3): track 10.5 -> 22.2 mm
- net Net-(MC3-Pin_3): track 12.5 -> 24.0 mm
- net Net-(MC4-Pin_2): track 10.6 -> 21.9 mm
- net Net-(MC3-Pin_7): track 30.2 -> 20.2 mm
- net Net-(MC1-Pin_6): track 10.5 -> 19.0 mm
- net Net-(MC1-Pin_7): track 14.1 -> 22.6 mm
- net Net-(MC4-Pin_5): track 17.3 -> 10.1 mm
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- removed copper zone on In2.Cu, net original5V
Other:
- board text added: "resistor"
- board text removed: "100k"
- board text removed: "D G S"
- board text removed: "NMOS"
- board text removed: "PMOS"
- board text removed: "resistors"
