File: Drill_ElevatorPCB/Drill_ElevatorPCB.kicad_sch (KiCad schematic)
At the start: 22 parts, among them J1 Barrel_Jack, J1 Conn_01x04_Socket, J2 Conn_01x04_Socket, J3 Conn_01x04_Socket, J4 Conn_01x04_Socket, SW1 SW_DIP_x01, SW10 SW_DIP_x01, SW11 SW_DIP_x01, SW12 SW_DIP_x01, SW2 SW_DIP_x01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

Commit message: schematicDone
Parts:
- added C2: C_Polarized, symbol Device:C_Polarized
Connections:
- net +12V: now also U1.16 (VMOT), U2.16 (VMOT), U3.16 (VMOT), U4.16 (VMOT), C2.1
- net GND: no longer J1.2
- net at J2.1 (Pin_1): now also U2.12 (A1)
- net at J2.2 (Pin_2): now also U2.11 (A2)
- net at J2.3 (Pin_3): now also U2.13 (B1)
- net at J2.4 (Pin_4): now also U2.14 (B2)
- net at J4.1 (Pin_1): now also U4.12 (A1)
- net at J4.2 (Pin_2): now also U4.11 (A2)
- net at J4.3 (Pin_3): now also U4.13 (B1)
- net at J4.4 (Pin_4): now also U4.14 (B2)
- net GND2: now reaches U4.15 (GND_MOT)
- net GND2: now also J1.2, U1.15 (GND_MOT), U2.15 (GND_MOT), U3.15 (GND_MOT), C2.2
- net at U1.11 (A2): now also J1.2 (Pin_2)
- net at U1.12 (A1): now also J1.1 (Pin_1)
- net at U1.13 (B1): now also J1.3 (Pin_3)
- net at U1.14 (B2): now also J1.4 (Pin_4)
- net at J3.1 (Pin_1): now also U3.12 (A1)
- net at J3.2 (Pin_2): now also U3.11 (A2)
- net at J3.3 (Pin_3): now also U3.13 (B1)
- net at J3.4 (Pin_4): now also U3.14 (B2)
Other:
- title: (none) -> Stepper Driver Board
- moved on the sheet: J1, J2, J3, J4

Commit message: Finalized schematic
Parts:
- added J5: Conn_01x02_Socket, symbol Connector:Conn_01x02_Socket
Connections:
- net +3.3V: now also U1.30 (VIN), J5.1 (Pin_1)
- net GND: now also J5.2 (Pin_2)

Commit message: foot prints assigend
Parts:
- C2: footprint (none) -> Capacitor_THT:CP_Radial_Tantal_D5.0mm_P5.00mm
- J1, J2, J3, J4: footprint (none) -> Connector_PinHeader_1.00mm:PinHeader_1x04_P1.00mm_Vertical
- J5: footprint (none) -> Connector_PinHeader_1.00mm:PinHeader_1x02_P1.00mm_Vertical
- J6: renamed from J1; footprint (none) -> Connector_BarrelJack:BarrelJack_Horizontal
- SW1, SW10, SW11, SW12, SW2, SW3, SW4, SW5, SW6, SW7, SW8, SW9: footprint (none) -> Button_Switch_THT:SW_DIP_SPSTx01_Slide_9.78x4.72mm_W7.62mm_P2.54mm
- U1, U2, U3, U4: footprint DRV8825_STEPPER_MOTOR_DRIVER_CARRIER:IC_DRV8825_STEPPER_MOTOR_DRIVER_CARRIER -> hi:IC_DRV8825_STEPPER_MOTOR_DRIVER_CARRIER
- U5: renamed from U1; footprint ESP32-DEVKIT-V1:MODULE_ESP32_DEVKIT_V1 -> hi:MODULE_ESP32_DEVKIT_V1
Changed lines of the file:
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@@
 			)
 		)
-		(property "Footprint" ""
+		(property "Footprint" "Connector_PinHeader_1.00mm:PinHeader_1x04_P1.00mm_Vertical"
 			(at 278.13 46.99 0)
 			(effects
@@
 			)
 		)
-		(property "Footprint" ""
+		(property "Footprint" "Connector_PinHeader_1.00mm:PinHeader_1x04_P1.00mm_Vertical"
 			(at 177.8 39.37 0)
 			(effects
@@
 			)
 		)
-		(property "Footprint" "DRV8825_STEPPER_MOTOR_DRIVER_CARRIER:IC_DRV8825_STEPPER_MOTOR_DRIVER_CARRIER"
+		(property "Footprint" "hi:IC_DRV8825_STEPPER_MOTOR_DRIVER_CARRIER"
 			(at 139.7 39.37 0)
 			(effects
@@
 			)
 		)
-		(property "Footprint" ""
+		(property "Footprint" "Button_Switch_THT:SW_DIP_SPSTx01_Slide_9.78x4.72mm_W7.62mm_P2.54mm"
 			(at 104.14 140.97 0)
 			(effects
@@
 			)
 		)
-		(property "Footprint" "DRV8825_STEPPER_MOTOR_DRIVER_CARRIER:IC_DRV8825_STEPPER_MOTOR_DRIVER_CARRIER"
+		(property "Footprint" "hi:IC_DRV8825_STEPPER_MOTOR_DRIVER_CARRIER"
 			(at 228.6 119.38 0)
 			(effects
@@
 		(dnp no)
 		(fields_autoplaced yes)
-		(property "Reference" "J1"
+		(property "Reference" "J6"
 			(at 30.48 19.05 0)
 			(effects
@@
 			)
 		)
-		(property "Footprint" ""
+		(property "Footprint" "Connector_BarrelJack:BarrelJack_Horizontal"
 			(at 31.75 28.956 0)
 			(effects
@@
 			(project ""
 				(path "/bee8b314-4813-4266-b002-9a06a0a76faa"
-					(reference "J1")
+					(reference "J6")
 					(unit 1)
 				)
@@
 			)
 		)
-		(property "Footprint" ""
+		(property "Footprint" "Button_Switch_THT:SW_DIP_SPSTx01_Slide_9.78x4.72mm_W7.62mm_P2.54mm"
 			(at 215.9 60.96 0)
 			(effects
@@
 			)
 		)
-		(property "Footprint" ""
+		(property "Footprint" "Connector_PinHeader_1.00mm:PinHeader_1x04_P1.00mm_Vertical"
 			(at 163.83 124.46 0)
 			(effects
@@
 			)
 		)
-		(property "Footprint" "DRV8825_STEPPER_MOTOR_DRIVER_CARRIER:IC_DRV8825_STEPPER_MOTOR_DRIVER_CARRIER"
+		(property "Footprint" "hi:IC_DRV8825_STEPPER_MOTOR_DRIVER_CARRIER"
 			(at 135.89 124.46 0)
 			(effects
@@
 		(dnp no)
 		(fields_autoplaced yes)
-		(property "Reference" "U1"
+		(property "Reference" "U5"
 			(at 49.53 44.45 0)
 			(effects
@@
 			)
 		)
-		(property "Footprint" "ESP32-DEVKIT-V1:MODULE_ESP32_DEVKIT_V1"
+		(property "Footprint" "hi:MODULE_ESP32_DEVKIT_V1"
 			(at 49.53 77.47 0)
 			(effects
@@
 			(project ""
 				(path "/bee8b314-4813-4266-b002-9a06a0a76faa"
-					(reference "U1")
+					(reference "U5")
 					(unit 1)
 				)
@@
 			)
 		)
-		(property "Footprint" ""
+		(property "Footprint" "Button_Switch_THT:SW_DIP_SPSTx01_Slide_9.78x4.72mm_W7.62mm_P2.54mm"
 			(at 104.14 129.54 0)
 			(effects
@@
 			)
 		)
-		(property "Footprint" ""
+		(property "Footprint" "Button_Switch_THT:SW_DIP_SPSTx01_Slide_9.78x4.72mm_W7.62mm_P2.54mm"
 			(at 196.85 146.05 0)
 			(effects
@@
 			)
 		)
-		(property "Footprint" ""
+		(property "Footprint" "Button_Switch_THT:SW_DIP_SPSTx01_Slide_9.78x4.72mm_W7.62mm_P2.54mm"
 			(at 104.14 151.13 0)
 			(effects
@@
 			)
 		)
-		(property "Footprint" ""
+		(property "Footprint" "Button_Switch_THT:SW_DIP_SPSTx01_Slide_9.78x4.72mm_W7.62mm_P2.54mm"
 			(at 196.85 124.46 0)
 			(effects
@@
 			)
 		)
-		(property "Footprint" ""
+		(property "Footprint" "Button_Switch_THT:SW_DIP_SPSTx01_Slide_9.78x4.72mm_W7.62mm_P2.54mm"
 			(at 215.9 49.53 0)
 			(effects
@@
 			)
 		)
-		(property "Footprint" ""
+		(property "Footprint" "Button_Switch_THT:SW_DIP_SPSTx01_Slide_9.78x4.72mm_W7.62mm_P2.54mm"
 			(at 107.95 55.88 0)
 			(effects
@@
 			)
 		)
-		(property "Footprint" ""
+		(property "Footprint" "Button_Switch_THT:SW_DIP_SPSTx01_Slide_9.78x4.72mm_W7.62mm_P2.54mm"
 			(at 107.95 44.45 0)
 			(effects
@@
 			)
 		)
-		(property "Footprint" ""
+		(property "Footprint" "Button_Switch_THT:SW_DIP_SPSTx01_Slide_9.78x4.72mm_W7.62mm_P2.54mm"
 			(at 196.85 135.89 0)
 			(effects
@@
 			)
 		)
-		(property "Footprint" ""
+		(property "Footprint" "Button_Switch_THT:SW_DIP_SPSTx01_Slide_9.78x4.72mm_W7.62mm_P2.54mm"
 			(at 215.9 71.12 0)
 			(effects
@@
 			)
 		)
-		(property "Footprint" ""
+		(property "Footprint" "Button_Switch_THT:SW_DIP_SPSTx01_Slide_9.78x4.72mm_W7.62mm_P2.54mm"
 			(at 107.95 66.04 0)
 			(effects
@@
 			)
 		)
-		(property "Footprint" ""
+		(property "Footprint" "Connector_PinHeader_1.00mm:PinHeader_1x04_P1.00mm_Vertical"
 			(at 261.62 119.38 0)
 			(effects
@@
 			)
 		)
-		(property "Footprint" ""
+		(property "Footprint" "Capacitor_THT:CP_Radial_Tantal_D5.0mm_P5.00mm"
 			(at 47.9552 30.48 0)
 			(effects
@@
 			)
 		)
-		(property "Footprint" "DRV8825_STEPPER_MOTOR_DRIVER_CARRIER:IC_DRV8825_STEPPER_MOTOR_DRIVER_CARRIER"
+		(property "Footprint" "hi:IC_DRV8825_STEPPER_MOTOR_DRIVER_CARRIER"
 			(at 247.65 44.45 0)
 			(effects
@@
 			)
 		)
-		(property "Footprint" ""
+		(property "Footprint" "Connector_PinHeader_1.00mm:PinHeader_1x02_P1.00mm_Vertical"
 			(at 81.28 19.05 0)
 			(effects

Commit message: PCB
Connections:
- net SLP/RST 1: now also U5.20 (D35); no longer U5.5 (D4)
- net SLP/RST 2: now also U5.19 (D34); no longer U5.8 (D5)
- net SLP/RST 3: now also U5.11 (D21); no longer U5.27 (D12)
- net SLP/RST 4: now also U5.25 (D27); no longer U5.28 (D13)
- net dir_1: now also U5.21 (D32); no longer U5.26 (D14)
- net dir_2: now also U5.26 (D14); no longer U5.3 (D15)
- net dir_4: now also U5.24 (D26); no longer U5.10 (D19)
- net step_1: now also U5.22 (D33); no longer U5.11 (D21)
- net step_2: now also U5.28 (D13); no longer U5.14 (D22)
- net step_3: now also U5.10 (D19); no longer U5.15 (D23)
- net at J2.1 (Pin_1): now also U2.11 (A2); no longer U2.12 (A1)
- net at J2.2 (Pin_2): now also U2.12 (A1); no longer U2.11 (A2)
- net at J4.1 (Pin_1): now also U4.11 (A2); no longer U4.12 (A1)
- net at J4.2 (Pin_2): now also U4.12 (A1); no longer U4.11 (A2)
- net at U1.11 (A2): now also J1.1 (Pin_1); no longer J1.2 (Pin_2)
- net at U1.12 (A1): now also J1.2 (Pin_2); no longer J1.1 (Pin_1)
- net at J3.1 (Pin_1): now also U3.11 (A2); no longer U3.12 (A1)
- net at J3.2 (Pin_2): now also U3.12 (A1); no longer U3.11 (A2)
