File: Drill_ElevatorPCB/Drill_ElevatorPCB.kicad_pcb (KiCad board)
At the start: 2 copper layers, 24 parts, among them J1 Conn_01x04_Socket, J2 Conn_01x04_Socket, J3 Conn_01x04_Socket, J4 Conn_01x04_Socket, J5 Conn_01x02_Socket, J6 Barrel_Jack, SW1 SW_DIP_x01, SW10 SW_DIP_x01, SW11 SW_DIP_x01, SW12 SW_DIP_x01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

Commit message: PCB
Parts:
- moved J6 103.8 mm to (102.5, 65.8), turned to -90 degrees
- moved J5 101.0 mm to (121.7, 57.4), turned to -90 degrees
- moved U3 100.9 mm to (108.0, 138.4), turned to 180 degrees
- moved C2 99.1 mm to (112.0, 65.3), turned to 90 degrees
- moved J2 95.6 mm to (99.0, 80.6)
- moved SW10 86.5 mm to (126.1, 144.2), turned to 180 degrees
- moved J3 85.6 mm to (98.7, 136.0)
- moved SW11 81.2 mm to (126.1, 138.9), turned to 180 degrees
- moved SW12 77.1 mm to (126.2, 133.4), turned to 180 degrees
- moved SW9 74.5 mm to (127.1, 80.3), turned to 180 degrees
- moved SW5 73.6 mm to (130.9, 138.7)
- moved SW6 73.0 mm to (131.0, 144.2)
- moved SW8 67.5 mm to (127.2, 85.8), turned to 180 degrees
- moved SW7 63.7 mm to (127.1, 91.5), turned to 180 degrees
- moved U2 63.7 mm to (108.5, 83.2), turned to 180 degrees
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Connections:
- U1 pad 11: Net-(J1-Pin_2) -> Net-(J1-Pin_1)
- U1 pad 12: Net-(J1-Pin_1) -> Net-(J1-Pin_2)
- U2 pad 11: Net-(J2-Pin_2) -> Net-(J2-Pin_1)
- U2 pad 12: Net-(J2-Pin_1) -> Net-(J2-Pin_2)
- U3 pad 11: Net-(J3-Pin_2) -> Net-(J3-Pin_1)
- U3 pad 12: Net-(J3-Pin_1) -> Net-(J3-Pin_2)
- U4 pad 11: Net-(J4-Pin_2) -> Net-(J4-Pin_1)
- U4 pad 12: Net-(J4-Pin_1) -> Net-(J4-Pin_2)
- U5 pad 10: dir_4 -> step_3
- U5 pad 11: step_1 -> SLP/RST 3
- U5 pad 14: step_2 -> unconnected-(U5-D22-Pad14)
- U5 pad 15: step_3 -> unconnected-(U5-D23-Pad15)
- U5 pad 19: unconnected-(U5-D34-Pad19) -> SLP/RST 2
- U5 pad 20: unconnected-(U5-D35-Pad20) -> SLP/RST 1
- U5 pad 21: unconnected-(U5-D32-Pad21) -> dir_1
- U5 pad 22: unconnected-(U5-D33-Pad22) -> step_1
- U5 pad 24: unconnected-(U5-D26-Pad24) -> dir_4
- U5 pad 25: unconnected-(U5-D27-Pad25) -> SLP/RST 4
- U5 pad 26: dir_1 -> dir_2
- U5 pad 27: SLP/RST 3 -> unconnected-(U5-D12-Pad27)
- U5 pad 28: SLP/RST 4 -> step_2
- U5 pad 3: dir_2 -> unconnected-(U5-D15-Pad3)
- U5 pad 5: SLP/RST 1 -> unconnected-(U5-D4-Pad5)
- U5 pad 8: SLP/RST 2 -> unconnected-(U5-D5-Pad8)
Routing:
- net GND2: track 0.00 -> 284.8 mm
- net +12V: track 0.00 -> 252.1 mm, vias 0 -> 1
- net GND: track 0.00 -> 200.8 mm, vias 0 -> 1
- net +3.3V: track 0.00 -> 122.8 mm
- net dir_1: track 0.00 -> 63.6 mm
- net step_1: track 0.00 -> 56.5 mm
- net SLP/RST 1: track 0.00 -> 54.4 mm
- net SLP/RST 2: track 0.00 -> 35.4 mm
- net SLP/RST 3: track 0.00 -> 33.3 mm
- net SLP/RST 4: track 0.00 -> 28.7 mm
- net dir_2: track 0.00 -> 27.7 mm
- net step_3: track 0.00 -> 24.6 mm
- net step_2: track 0.00 -> 23.9 mm
- net dir_3: track 0.00 -> 21.0 mm
- net Net-(U4-M2): track 0.00 -> 11.1 mm
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
Commit message: hello
Routing:
- net GND: track 200.8 -> 226.2 mm
Changed lines of the file:
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@@
+	)
+	(segment
+		(start 115.05 98.15)
+		(end 115.05 123.55)
+		(width 0.2)
+		(layer "F.Cu")
+		(net 19)
 	)
 	(segment
